Commit message: update urdf to point to correct mesh location

File: urdf/_d435.urdf.xacro (robot description, xacro)
@@ -48,5 +48,5 @@
         <geometry>
           <!-- <box size="${d435_cam_width} ${d435_cam_height} ${d435_cam_depth}"/> -->
-          <mesh filename="package://dynus/share/dynus/meshes/real_sense/d435.dae" />
+          <mesh filename="$(find dynus)/meshes/real_sense/d435.dae" />
         </geometry>
         <material name="${name}_aluminum"/>
